Commit message: added Dabai

File: src/my_robot_description/urdf/rubot/rubot_mecanum.urdf (robot description, URDF)
Before this commit: robot rubot, 9 links, 8 joints
Links:
- removed link camera
Joints:
- removed joint joint_camera

Commit message: urdf depth

File: src/my_robot_description/urdf/rubot/rubot_mecanum.urdf (robot description, URDF)
Before this commit: robot rubot, 8 links, 7 joints
Links:
- added link camera, mass 0.01; collision box size=0.025 0.05 0.025; visual box size=0.025 0.05 0.025
Joints:
- added joint joint_camera: type fixed, parent base_link, child camera, origin xyz=0.130 0.0 0.08 rpy=0 0 0
