Commit message: depth

File: src/my_robot_description/urdf/rubot/rubot_mecanum_gz.urdf (robot description, URDF)
Before this commit: robot rubot_mecanum, 8 links, 7 joints
Links:
- removed link camera_link
- added link camera; visual box size=0.025 0.05 0.025
Joints:
- joint camera_joint: child camera_link -> camera
