Commit message: Number 2 mesh added to rubot

File: src/my_robot_description/urdf/rubot/rubot_grup1.urdf (robot description, URDF)
Before this commit: robot rubot_mecanum, 8 links, 7 joints
Links:
- removed link camera
- added link top_part, mass 0.2; collision box size=0.12 0.12 0.06; visual mesh filename=package://my_robot_description/meshes/rubot/number2.stl scale=0.001 0.001 0.001
Joints:
- removed joint camera_joint
- added joint top_part_joint: type fixed, parent base_link, child top_part, origin xyz=0 0 0.20 rpy=0 0 0
