Commit message: Practica 2

File: src/my_robot_description/urdf/rubot/rubot_grup2.urdf (robot description, URDF)
Before this commit: robot rubot_mecanum, 9 links, 8 joints
Links:
- removed link top_part
- added link lidar_cube, mass 0.005; collision box size=0.02 0.02 0.02; visual box size=0.03 0.03 0.03
- added link part, mass 0.01; collision box size=0.05 0.05 0.025; visual mesh filename=file://$(find my_robot_description)/meshes/rubot/number2.stl scale=0.0008 0.0008 0.0008
- link base_link: geometry collision box size=0.23 0.12 0.1; visual mesh filename=file://$(find my_robot_description)/meshes/rubot/base_link.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 scale=0.001 0.001 0.001
Joints:
- added joint lidar_cube_joint: type fixed, parent base_scan, child lidar_cube, origin xyz=0 0 0.005 rpy=0 0 0
- joint joint_part: child top_part -> part; origin xyz=0 0 0.20 rpy=0 0 0 -> xyz=-0.10 0.0 0.08 rpy=0 0 0
- joint upper_left_wheel_joint: origin xyz=0.07 0.10 0.00 rpy=0 0 0 -> xyz=0.07 0.1 0 rpy=0 0 0
